File: hw/misc.kicad_sch (KiCad schematic)
At the start: 4 parts

Commit message: 1p version
Parts:
- removed H1, H2, H3, H4: MountingHole, MountingHole:MountingHole_2.2mm_M2, symbol Mechanical:MountingHole
Other:
- note removed: "Mounting Holes"
