File: hw/c64_controls_sch.kicad_sch (KiCad schematic)
At the start: 12 parts, among them J300 DE9_Receptacle, J301 DE9_Receptacle, U300 74AHCT1G125, U301 74AHCT1G125, U302 74AHCT1G125, U303 74AHCT1G125, U304 74AHCT1G125, U305 74AHCT1G125, U306 74AHCT1G125, U307 74AHCT1G125, U308 74AHCT1G125, U309 74AHCT1G125

Commit message: rerouted
Parts:
- added C300, C301, C302, C303, C304, C305, C306, C307, C308, C309: 100n, Capacitor_SMD:C_0402_1005Metric, symbol Device:C
Connections:
- net GND: now also C300.2, C301.2, C302.2, C303.2, C304.2, C305.2, C306.2, C307.2, C308.2, C309.2
- net VBUS: now also C300.1, C301.1, C302.1, C303.1, C304.1, C305.1, C306.1, C307.1, C308.1, C309.1

Commit message: 1p version
Parts:
- removed C305, C306, C307, C308, C309: 100n, Capacitor_SMD:C_0402_1005Metric, symbol Device:C
- removed J301: DE9_Receptacle, Connector_Dsub:DSUB-9_Female_Horizontal_P2.77x2.84mm_EdgePinOffset4.94mm_Housed_MountingHolesOffset4.94mm, symbol Connector:DE9_Receptacle
- removed U305, U306, U307, U308, U309: 74AHCT1G125, Package_TO_SOT_SMD:SOT-353_SC-70-5, symbol 74xGxx:74AHCT1G125
- J300: footprint Connector_Dsub:DSUB-9_Female_Horizontal_P2.77x2.84mm_EdgePinOffset4.94mm_Housed_MountingHolesOffset4.94mm -> Connector_Dsub:DSUB-9_Female_EdgeMount_P2.77mm
Connections:
- no-connect marks 8 -> 4
Other:
- note removed: "Joystick 2 Buffers"
- moved on the sheet: C300, C301, C302, C303, C304, J300, U300, U301, U302, U303, U304

Commit message: pre production review
Connections:
- net GND: now also J300.8
- net VBUS renamed +5V
- no-connect marks 4 -> 3
Other:
- moved on the sheet: C300, U300
