File: hw/usb-64-rev2c.kicad_pcb (KiCad board)
At the start: 4 copper layers, 24.5 x 41 mm, 51 parts, among them IC1 NCP708MU330TAG, J1 USB_C_Receptacle_PowerOnly_6P, J100 Conn_01x05_Pin, J2 USB_A, J300 DE9_Receptacle, SW1 SW_Push, U200 RP2040, U201 W25Q16JVUXIQ, U300 74AHCT1G125, U301 74AHCT1G125, U302 74AHCT1G125, U303 74AHCT1G125, U304 74AHCT1G125, X100 ASE-12MHz

Commit message: pre production review
Parts:
- removed D1: ESD7L5.0DT5G, Package_TO_SOT_SMD:SOT-723
- removed IC1: NCP708MU330TAG, Package_SON:SON95P300X300X55-7N
- added H1: MountingHole, MountingHole:MountingHole_2.2mm_M2, F.Cu at (160.5, 93.2)
- added U1: TPD2EUSB30, Package_TO_SOT_SMD:Texas_DRT-3, F.Cu at (155.2, 83.4)
- added U2: TLV76733DRVx, Package_SON:WSON-6-1EP_2x2mm_P0.65mm_EP1x1.6mm_ThermalVias, F.Cu at (146.3, 86.0)
- C1: value 1u -> 10n; footprint Capacitor_SMD:C_0603_1608Metric -> Capacitor_SMD:C_0402_1005Metric
- C2: value 1u -> 100n
- C3: value 4.7u -> 1u; footprint Capacitor_SMD:C_1206_3216Metric -> Capacitor_SMD:C_0603_1608Metric
- C4: value 4.7u -> 10u; footprint Capacitor_SMD:C_1206_3216Metric -> Capacitor_SMD:C_0805_2012Metric
- R6, R9: value 330 -> 1k
- moved D2 5.01 mm to (154.1, 86.7), turned to -90 degrees
- moved C2 4.52 mm to (150.9, 85.1)
- moved C1 3.86 mm to (151.8, 88.1), turned to 180 degrees
- moved C3 2.46 mm to (148.5, 85.8)
- moved FB1 2.19 mm to (151.1, 86.7), turned to 180 degrees
- moved R6 1.97 mm to (142.1, 90.5), turned to 180 degrees
- moved D6 1.49 mm to (143.8, 89.6)
- moved J100 0.60 mm to (140.8, 77.5)
- moved R204 0.50 mm to (160.2, 73.0)
- moved R203 0.50 mm to (160.2, 72.0)
- moved C302 0.30 mm to (153.0, 61.5)
- moved C4 0.20 mm to (144.0, 86.3), turned to -90 degrees
- moved R8 0.20 mm to (144.8, 92.9)
- moved R7 0.13 mm to (156.6, 92.9)
- moved C208 0.13 mm to (145.9, 76.3)
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- renumbered FB3 to FB1
Connections:
- C1 pad 1: Net-(C1-Pad1) -> VBUS
- C2 pad 1: VBUS -> +5V
- C3 pad 1: VBUS -> +5V
- C300 pad 1: VBUS -> +5V
- C301 pad 1: VBUS -> +5V
- C302 pad 1: VBUS -> +5V
- C303 pad 1: VBUS -> +5V
- C304 pad 1: VBUS -> +5V
- FB1 pad 1: Net-(C1-Pad1) -> VBUS
- FB1 pad 2: VBUS -> +5V
- J1 pad A9: Net-(C1-Pad1) -> VBUS
- J1 pad B9: Net-(C1-Pad1) -> VBUS
- J300 pad 8: unconnected-(J300-Pad8) -> GND
- U300 pad 5: VBUS -> +5V
- U301 pad 5: VBUS -> +5V
- U302 pad 5: VBUS -> +5V
- U303 pad 5: VBUS -> +5V
- U304 pad 5: VBUS -> +5V
Routing:
- net +5V: track 0.00 -> 76.8 mm, vias 0 -> 6
- net VBUS: track 76.4 -> 11.1 mm, vias 6 -> 0
- net Net-(C1-Pad1): track 10.1 -> 0.00 mm
- net /USB_MCU_D_P: track 25.6 -> 19.1 mm
- net /USB_MCU_D_N: track 25.3 -> 18.8 mm
- net GND: track 53.8 -> 59.8 mm, vias 83 -> 94
- net Net-(D2-K): track 7.81 -> 2.44 mm
- net +3.3V: track 102.1 -> 97.1 mm, vias 4 -> 5
- net +1V1: track 24.8 -> 29.4 mm
- net /MCU/SWD: track 14.9 -> 16.4 mm
- net /MCU/UART_TX: track 13.6 -> 14.8 mm
- net /C64_controls/IO_DOWN: track 12.5 -> 13.1 mm
- net /MCU/SWCLK: track 12.8 -> 13.4 mm
- net /MCU/UART_RX: track 13.4 -> 14.0 mm
- net /MCU/MCU_QSPI_SS: track 15.8 -> 15.2 mm
Other:
- board text removed: "CLK"
- board text removed: "CS"
- board text removed: "D"
- board text removed: "G"
- board text removed: "PWR"
- board text removed: "RX"
- board text removed: "TX"

Commit message: production
Parts:
- U200: footprint Package_DFN_QFN:QFN-56-1EP_7x7mm_P0.4mm_EP3.2x3.2mm -> Package_DFN_QFN:QFN-56-1EP_7x7mm_P0.4mm_EP3.2x3.2mm_ThermalVias
- moved C202 0.71 mm to (148.9, 79.6)
- moved C203 0.10 mm to (147.9, 78.8)
- moved C215 0.07 mm to (152.2, 69.0)
- moved X100 0.07 mm to (153.1, 67.2)
Routing:
- net +3.3V: track 97.1 -> 69.5 mm, vias 5 -> 4
- net GND: track 59.8 -> 53.6 mm, vias 94 -> 86
- net +1V1: track 29.4 -> 31.2 mm
- added copper zone on F.Cu, net +3.3V
